Commit message: feat: package the current research pipeline and handoff docs

File: assets/robots/onrobot_rg6/onrobot_rg6.urdf (robot description, URDF)
Before this commit: robot onrobot_rg6_model, 7 links, 6 joints
Links:
- link left_inner_finger: geometry collision mesh filename=meshes/collision/inner_finger.stl; visual mesh filename=meshes/visual/inner_finger.stl
- link left_inner_knuckle: geometry collision mesh filename=meshes/collision/inner_knuckle.stl; visual mesh filename=meshes/visual/inner_knuckle.stl
- link left_outer_knuckle: geometry collision mesh filename=meshes/collision/outer_knuckle.stl; visual mesh filename=meshes/visual/outer_knuckle.stl
- link onrobot_rg6_base_link: geometry collision mesh filename=meshes/collision/base_link.stl; visual mesh filename=meshes/visual/base_link.stl
- link right_inner_finger: geometry collision mesh filename=meshes/collision/inner_finger.stl; visual mesh filename=meshes/visual/inner_finger.stl
- link right_inner_knuckle: geometry collision mesh filename=meshes/collision/inner_knuckle.stl; visual mesh filename=meshes/visual/inner_knuckle.stl
- link right_outer_knuckle: geometry collision mesh filename=meshes/collision/outer_knuckle.stl; visual mesh filename=meshes/visual/outer_knuckle.stl
